File: Hardware/RFBoard.sch (EAGLE design)
At the start: 188 parts, among them IC1 HMC1097, IC10 NCP702-1.8, IC11 QPC6082, IC12 MCP4812, IC13 QPC6082, IC2 MAX2871, IC3 AP2114HA-3.3, IC4 NCP702-3.3, IC5 NCP702-3.3, IC6 MAX5873, IC7 NCP702-1.8, IC8 NCP702-3.3, IC9 NCP702-3.3

Commit message: Heterodyne path sheet
Parts:
- added C101, C119: 10n, rcl:C-EUC0603
- added C102, C104: 820p, rcl:C-EUC0603
- added C103, C113, C114, C115, C118: 100n, rcl:C-EUC0603
- added C105, C110: 10u, rcl:C-EUC0603
- added C106, C107: 5p6, rcl:C-EUC0603
- added C108, C109, C120: DNP, rcl:C-EUC0603
- added C111, C112, C116, C117, C121, C122, C123, C124, C125: 1u, rcl:C-EUC0603
- added IC14: LT5560, rf:LT5560
- added IC15: ADF4360, rf:ADF4360
- added IC16, IC17: HMC284, rf:HMC284
- added IC18, IC19: NCP702-3.3, rf:NCP702
- added IC20: LT1395, linear:OPA344N-SOT23
- added L50, L51: 100n, rf:INDUCTOR0603
- added L52, L53, L54, L55: 3n9, rf:INDUCTOR0603
- added L56: (no value), rcl:L-EUL2012C
- added Q1, Q2: BSS123, transistor-small-signal:BSS123
- added R27: 250, resistor:R-EU_R0603
- added R28: 470, rcl:R-EU_R0603
- added R29: 120, resistor:R-EU_R0603
- added R30, R41, R42: 4k7, resistor:R-EU_R0603
- added R31, R32: 10k, resistor:R-EU_R0603
- added R33: 3, resistor:R-EU_R0603
- added R34: 0, resistor:R-EU_R0603
- added R35, R36: DNP, resistor:R-EU_R0603
- added R37, R38, R39, R40: 200, resistor:R-EU_R0603
- added R43: 49R9, rcl:R-EU_R0603
- added U$1: HHM1522B1, rf:HHM1522B1
- C19: value 10n -> 100n
Connections:
- removed net OFFSET_SCK: IC12.SCK
- removed net OFFSET_SDI: IC12.SDI
- removed net SYNTH_CLK: R5.1
- removed net SYNTH_DATA: R6.1
- removed net SYNTH_REF: C19.1
- new net 10MHZ_REF: C115.2, C19.1
- new net ADF_CE: IC15.CE
- new net ADF_LE: IC15.LE
- new net ADF_MUX: IC15.MUXOUT
- new net DAC_DIG3.1: C105.1, C111.1, C113.1, C114.1, IC15.AVDD, IC15.DVDD, IC15.VVCO, IC18.VOUT, L50.1, L51.1
- new net DAC_DIG3.2: C116.1, C118.1, IC14.VCC, IC19.VOUT, R37.2, R38.2
- new net EN_HETERODYNE: Q1.G
- new net FULLBAND: IC17.RFC
- new net MIX_EN: IC14.EN
- new net N$100: C109.1, IC14.LO+, L52.1
- new net N$101: C109.2, IC14.LO-, L53.1
- new net N$102: C119.1, IC16.RFC
- new net N$103: IC12.VB, R28.1
- new net N$104: C120.2, L54.2, U$1.+
- new net N$105: IC14.IN+, L54.1
- new net N$106: IC14.IN-, L55.1
- new net N$107: C120.1, L55.2, U$1.-
- new net N$108: IC16.RF2, IC17.RF1
- new net N$109: IC16.RF1, R34.2, R35.1
- new net N$110: R33.1, U$1.DC
- new net N$111: R34.1, R36.1, U$1.UN
- new net N$112: C121.1, IC20.V+, L56.1
- new net N$113: C122.1, IC14.OUT+, R37.1
- new net N$114: C123.2, IC14.OUT-, R38.1
- new net N$115: C125.2, IC20.OUT, R39.1
- new net N$116: C123.1, IC20.-IN, R39.2
- new net N$117: C122.2, IC20.+IN, R40.2
- new net N$118: C124.2, R40.1, R41.1, R42.1
- new net N$119: C125.1, R43.1
- new net N$120: IC17.RF2, R43.2
- new net N$86: IC15.RSET, R30.2
- new net N$87: C101.1, IC15.CC
- new net N$88: C102.1, R29.2
- new net N$92: C103.1, IC15.CP, R27.1, R29.1
- new net N$93: C104.1, IC15.VTUNE, R27.2
- new net N$94: C115.1, IC15.REFIN
- new net N$95: C105.2, IC15.CN
- new net N$96: C106.1, IC15.RFOUTA, L50.2
- new net N$97: C107.2, IC15.RFOUTB, L51.2
- new net N$98: C106.2, C108.1, L52.2
- new net N$99: C107.1, C108.2, L53.2
- new net SPI_CLK: IC12.SCK, IC15.CLK, R5.1
- new net SPI_MOSI: IC12.SDI, IC15.DATA, R6.1
- new net SW_DIRECT: IC16.A, IC17.B, Q1.D, Q2.G, R31.2
- new net SW_HET: IC16.B, IC17.A, Q2.D, R32.2
- net +5V: now also C112.1, C117.1, IC18.EN, IC18.VIN, IC19.EN, IC19.VIN, L56.2, R31.1, R32.1, R41.2
- net FILTERED: now also C119.2
- net GND: now also C101.2, C102.2, C103.2, C104.2, C110.2, C111.2, C112.2, C113.2, C114.2, C116.2, C117.2, C118.2, C121.2, C124.1, C55.2, IC14.GND, IC15.AGND, IC15.CPGND, IC15.DGND, IC16.GND, IC17.GND, IC18.GND, IC19.GND, IC20.V-, Q1.S, Q2.S, R30.1, R33.2, R35.2, R36.2, R42.2, U$1.GND
- net N$30: now also C110.1, R28.2
Other:
- note added: "-3dbm@250MHz, -6dbm@3GHz, -8dbm@6GHz"
- note added: "-4dbm@250MHz, -8dbm@3GHz, -10dbm@6GHz"
- note added: "0.1-3GHz: approx. -2dbm output power"
- note added: "Heterodyne path"
- note removed: "0.1-3GHz: approx. 2dbm output power"

Commit message: RF part of schematic finished, placed most components on PCB
Parts:
- added C126, C127: 22p, rcl:C-EUC0603
- added C128, C129: 33p, rcl:C-EUC0603
- added C130, C131, C132, C133, C134, C135, C137, C138, C139, C142, C143, C144, C147, C148, C149, C150, C152, C153, C154, C155, C156, C157, C158: 1u, rcl:C-EUC0603
- added C136, C141, C146: 10n, rcl:C-EUC0603
- added C140, C145: 100p, rcl:C-EUC0603
- added C151: 1n, rcl:C-EUC0603
- added IC21, IC22, IC23: MAADSS0008, rf:MAADSS0008
- added IC24: RFSA2033, rf:RFSA2033
- added IC25, IC26: MMG3H21NT1, rf:HMC480
- added IC27: HMC1021, rf:HMC1021
- added IC28: MCP4812, dac:MCP4812
- added IC29, IC30: NCP702-3.3, rf:NCP702
- added L57, L67: (no value), rcl:L-EUL2012C
- added L58, L59, L60, L61, L64: 30n, rf:INDUCTOR0603
- added L62, L65: 470n, rf:INDUCTOR0603
- added L63, L66: SRU5018-101, rf:INDUCTOR5018
- added Q3, Q4, Q5: BSS123, transistor-small-signal:BSS123
- added R44, R45, R46, R54, R55, R56, R57, R58, R61, R62, R63, R64: 10k, resistor:R-EU_R0603
- added R47, R48: 0, resistor:R-EU_R0603
- added R49, R50: 8R66, resistor:R-EU_R0603
- added R51: 110, resistor:R-EU_R0603
- added R52: 77R5, resistor:R-EU_R0603
- added R53: 49R9, rcl:R-EU_R0603
- added R59, R60, R65: DNP, resistor:R-EU_R0603
- added X1: out, rf:SMA_CONNECTOR
- C17: value 100n -> 1u
Connections:
- net DAC_DIG3.1 renamed PLL_DIG3
- net EN_HETERODYNE renamed EN_DIREKT
- removed net +3V3: C59.1, C60.1, IC11.VDD, IC13.VDD
- new net 15DB1: IC21.V2, Q3.G
- new net 15DB2: IC22.V2, Q4.G
- new net 15DB3: IC23.V2, Q5.G
- new net DBM_CS: IC28.CS
- new net DET_SCI1: IC27.SCI1, R58.1
- new net DET_SCI2: IC27.SCI2, R57.1
- new net DET_SCI3: IC27.SCI3, R55.2
- new net DET_SCI4: IC27.SCI4, R56.2
- new net DET_\EN: IC27.ENX, R54.2
- new net GAIN_CTRL: C154.1, IC24.VC, R63.2
- new net N$121: C126.2, L58.2, R43.2
- new net N$122: C129.2, L58.1, L59.2
- new net N$123: C128.2, L59.1, L60.2
- new net N$124: C131.1, IC21.GND
- new net N$125: C130.1, IC21.RF1
- new net N$126: C132.1, IC22.RF1
- new net N$127: IC21.V1, Q3.D, R44.2
- new net N$128: C133.1, IC22.GND
- new net N$129: IC22.V1, Q4.D, R45.2
- new net N$130: C134.1, IC23.RF1
- new net N$131: C135.1, IC23.GND
- new net N$132: IC23.V1, Q5.D, R46.2
- new net N$133: C134.2, IC22.RF2
- new net N$134: C132.2, IC21.RF2
- new net N$135: C119.2, IC24.RFOUT
- new net N$136: C136.1, IC24.RFIN
- new net N$137: C137.1, IC24.VDD, L57.1
- new net N$138: C139.2, IC25.OUT, L61.2
- new net N$139: C138.1, IC25.IN
- new net N$140: L61.1, L62.2
- new net N$141: L62.1, L63.2
- new net N$142: C144.2, IC26.OUT, L64.2
- new net N$143: C140.1, C141.1, C142.1, L63.1, R47.1
- new net N$144: C139.1, IC26.IN
- new net N$145: C145.1, C146.1, C147.1, L66.1, R48.1
- new net N$146: L64.1, L65.2
- new net N$147: L65.1, L66.2
- new net N$148: C138.2, IC23.RF2
- new net N$149: C144.1, R49.2
- new net N$150: R49.1, R50.2, R51.1
- new net N$151: C143.1, R50.1
- new net N$152: C149.1, R51.2, R52.1
- new net N$153: C143.2, X1.1
- new net N$154: C148.1, IC27.VCC, L67.1
- new net N$155: C149.2, IC27.INP
- new net N$156: C150.2, IC27.INN
- new net N$158: C153.1, R62.2, R63.1, R65.1
- new net N$159: C150.1, R53.2
- new net N$160: C151.1, IC27.COFSB
- new net N$161: C151.2, IC27.COFSA
- new net N$162: C155.1, IC27.VSET, R59.1, R60.2, R61.1
- new net N$163: IC27.RMSOUT, R60.1, R62.1
- new net N$164: IC24.SLOPE, R64.2
- new net SETDAC_VCC: C152.1, C17.1, IC28.VDD, IC29.VOUT
- new net STEPPED25: IC11.RF1, IC13.RF5
- new net STEPPED37: IC11.RF2, IC13.RF6
- new net SWITCHES_VCC: C157.1, C59.1, C60.1, IC11.VDD, IC13.VDD, IC30.VOUT
- net +5V: now also C156.1, C158.1, IC29.EN, IC29.VIN, IC30.EN, IC30.VIN, L57.2, L67.2, R44.1, R45.1, R46.1, R47.2, R48.2, R54.1, R55.1, R56.1
- net FILTERED: now also C136.2; no longer C119.2
- net FULLBAND: now also C130.2
- net GND: now also C126.1, C127.1, C128.1, C129.1, C131.2, C133.2, C135.2, C137.2, C140.2, C141.2, C142.2, C145.2, C146.2, C147.2, C148.2, C152.2, C153.2, C154.2, C155.2, C156.2, C157.2, C158.2, IC24.EN, IC24.GND, IC25.GND, IC26.GND, IC27.GND, IC28.LDAC, IC28.VSS, IC29.GND, IC30.GND, Q3.S, Q4.S, Q5.S, R52.2, R53.1, R57.2, R58.2, R59.2, R64.1, X1.2
- net N$10: no longer C17.1
- net N$105: now also IC28.VA, R61.2; no longer IC14.IN+, L54.1
- net N$106: now also IC28.VB, R65.2; no longer IC14.IN-, L55.1
- net N$108: now also IC16.RF1, IC17.RF2; no longer IC16.RF2, IC17.RF1
- net N$109: now also IC16.RF2; no longer IC16.RF1
- net N$12: now also IC2.RFOUTA_N; no longer IC2.RFOUTA_P
- net N$120: now also C127.2, IC17.RF1, L60.1; no longer IC17.RF2, R43.2
- net N$14: now also IC2.RFOUTA_P; no longer IC2.RFOUTA_N
- net N$52: now also IC11.RF3; no longer IC11.RF1
- net N$53: now also IC13.RF7; no longer IC13.RF5
- net N$60: now also IC11.RF4; no longer IC11.RF2
- net N$61: now also IC14.IN+, L55.1; no longer C70.1, IC13.RF6, L28.1
- net N$68: now also IC14.IN-, L54.1; no longer C77.1, IC11.RF3, L29.2
- net N$69: now also IC13.RF4; no longer IC13.RF7
- net N$76: now also IC11.RF7; no longer IC11.RF4
- net N$77: now also IC13.RF3; no longer IC13.RF8
- net N$84: now also IC11.RF6; no longer IC11.RF5
- net N$85: now also IC13.RF2; no longer IC13.RF1
- net N$89: now also IC11.RF5, IC13.RF1; no longer IC11.RF8, IC13.RF4
- net N$90: now also C77.1, IC11.RF8, L29.2; no longer IC11.RF7, IC13.RF3
- net N$91: now also C70.1, IC13.RF8, L28.1; no longer IC11.RF6, IC13.RF2
- net N$96: now also IC15.RFOUTB; no longer IC15.RFOUTA
- net N$97: now also IC15.RFOUTA; no longer IC15.RFOUTB
- net SPI_CLK: now also IC28.SCK
- net SPI_MOSI: now also IC28.SDI
Other:
- note added: "300MHz lowpass"
- note added: "63mA max"
- note added: "80mA"
- note added: "LQW18CNR47J00D"

Commit message: Almost all RF routing
Parts:
- removed C157, C158: 1u, rcl:C-EUC0603
- removed C22, C23, C24: 33p, rcl:C-EUC0603
- removed IC11, IC13: QPC6082, rf:QPC6082
- removed IC30: NCP702-3.3, rf:NCP702
- removed R15, R5, R6: 33, resistor:R-EU_R0603
- added IC31, IC32: QPC6064, rf:QPC6064
- added L68, L69: (no value), rcl:L-EUL2012C
Connections:
- removed net N$19: C22.2, IC2.CLK, R5.2
- removed net N$21: C24.2, IC2.LE, R15.2
- removed net N$24: C23.2, IC2.DATA, R6.2
- removed net N$89: IC11.RF5, IC13.RF1
- removed net STEPPED37: IC11.RF2, IC13.RF6
- new net ETOUT: IC27.ETOUT
- new net VDD2: C59.1, IC31.VDD, L68.2
- net +5V: now also L68.1, L69.1; no longer C158.1, IC30.EN, IC30.VIN
- net FILTERED: now also IC32.RFC; no longer IC13.RFC
- net GND: now also IC31.GND, IC31.VSS, IC32.GND, IC32.VSS; no longer C157.2, C158.2, C22.1, C23.1, C24.1, IC11.GND, IC13.GND, IC30.GND
- net MOD_OUT: now also IC31.RFC; no longer IC11.RFC
- net N$52: now also IC31.RF5; no longer IC11.RF3
- net N$53: now also IC32.RF2; no longer IC13.RF7
- net N$60: now also IC31.RF4; no longer IC11.RF4
- net N$69: now also IC32.RF4; no longer IC13.RF4
- net N$76: now also IC31.RF2; no longer IC11.RF7
- net N$77: now also IC32.RF5; no longer IC13.RF3
- net N$84: now also IC31.RF1; no longer IC11.RF6
- net N$85: now also IC32.RF6; no longer IC13.RF2
- net N$90: now also IC31.RF3; no longer IC11.RF8
- net N$91: now also IC32.RF3; no longer IC13.RF8
- net SPI_CLK: now also IC2.CLK; no longer R5.1
- net SPI_MOSI: now also IC2.DATA; no longer R6.1
- net STEPPED25: now also IC31.RF6, IC32.RF1; no longer IC11.RF1, IC13.RF5
- net SW1_CTL1: now also IC31.V1; no longer IC11.CTL1
- net SW1_CTL2: now also IC31.V2; no longer IC11.CTL2
- net SW1_CTL3: now also IC31.V3; no longer IC11.CTL3
- net SW2_CTL1: now also IC32.V1; no longer IC13.CTL1
- net SW2_CTL2: now also IC32.V2; no longer IC13.CTL2
- net SW2_CTL3: now also IC32.V3; no longer IC13.CTL3
- net SWITCHES_VCC: now also IC32.VDD, L69.2; no longer C157.1, C59.1, IC11.VDD, IC13.VDD, IC30.VOUT
- net SYNTH_LE: now also IC2.LE; no longer R15.1

Commit message: FPGA + power supply added
Parts:
- added C157, C163, C166, C167, C168, C169, C170, C171, C172, C173, C174: 100n, rcl:C-EUC0603
- added C158, C159, C164, C165: 22u, rcl:C-EUC1206
- added C160: 22p, rcl:C-EUC0603
- added C161, C23: 10n, rcl:C-EUC0603
- added C162, C24: 10u, rcl:C-EUC1206
- added C22: 1u, rcl:C-EUC0603
- added IC11: TPS42951, custom-ic:TPS42951
- added L70, L71: 2u2, custom-ic:SRN5040
- added R15, R5: 73k2, resistor:R-EU_R0603
- added R6, R66: 22k1, resistor:R-EU_R0603
- added R67: 22, resistor:R-EU_R0603
- added R68, R69, R70, R71: 10k, resistor:R-EU_R0603
- added SV1: (no value), con-ml:ML10
- added U1: 6SLX9TQG144, xilinx_devices_V6:6SLX9TQG144
- added U4: W25Q16BVSN, memory-winbond:W25Q16BVSN
Connections:
- new net +3V3: C158.1, C159.1, C160.1, C166.1, C167.1, C168.1, C169.1, C170.1, L70.2, R5.1, R68.2, R70.2, R71.2, SV1.4, U1B0.VCCO_0@0, U1B0.VCCO_0@1, U1B0.VCCO_0@2, U1B2.IO_L1N_M0_CMPMISO_2, U1B2.VCCO_2@0, U1B2.VCCO_2@1, U1BVCCAUX.VCCAUX@0, U1BVCCAUX.VCCAUX@1, U1BVCCAUX.VCCAUX@2, U1BVCCAUX.VCCAUX@3, U1BVCCAUX.VCCAUX@4, U4.!HOLD!, U4.!WP!, U4.VCC
- new net FLACH_MOSI: U1B2.IO_L3N_MOSI_CSI_B_MISO0_2, U4.DI
- new net FLASH_CLK: U1B2.IO_L1P_CCLK_2, U4.CLK
- new net FLASH_CS: U1B2.IO_L65N_CSO_B_2, U4.!CS!
- new net FLASH_MISO: R67.1, U4.DO
- new net N$165: C22.1, IC11VREG.VREG5
- new net N$166: C23.1, IC11G1.SS
- new net N$167: C160.2, IC11G1.VFB, R5.2, R6.1
- new net N$168: C161.1, IC11G2.SS
- new net N$169: C157.1, IC11G1.SW, L70.1
- new net N$170: C157.2, IC11G1.VBST
- new net N$171: IC11G2.VFB, R15.2, R66.1
- new net N$172: C163.1, IC11G2.SW, L71.1
- new net N$173: C163.2, IC11G2.VBST
- new net N$174: R67.2, U1B2.IO_L3P_D0_DIN_MISO_MISO1_2
- new net N$175: R70.1, U1B2.DONE_2
- new net N$176: R68.1, U1B2.PROGRAM_B_2
- new net N$177: R71.1, U1B2.IO_L65P_INIT_B_2
- new net N$19: SV1.3, U1BNA.TDO
- new net N$21: SV1.5, U1BNA.TMS
- new net N$24: SV1.9, U1BNA.TDI
- new net N$89: SV1.1, U1BNA.TCK
- new net VCCINT: C164.1, C165.1, C171.1, C172.1, C173.1, C174.1, L71.2, R15.1, U1BVCCINT.VCCINT@0, U1BVCCINT.VCCINT@1, U1BVCCINT.VCCINT@2, U1BVCCINT.VCCINT@3, U1BVCCINT.VCCINT@4
- net +5V: now also C162.1, C24.1, IC11G1.EN, IC11G1.VIN, IC11G2.EN, IC11G2.VIN
- net CLKN: now also U1B0.IO_L1N_VREF_0
- net CLKP: now also R69.2, U1B0.IO_L1P_HSWAPEN_0
- net GND: now also C158.2, C159.2, C161.2, C162.2, C164.2, C165.2, C166.2, C167.2, C168.2, C169.2, C170.2, C171.2, C172.2, C173.2, C174.2, C22.2, C23.2, C24.2, IC11G1.PGND, IC11G2.PGND, IC11VREG.GND, R6.2, R66.2, R69.1, SV1.10, SV1.2, U1B2.IO_L13P_M1_2, U1BGND.GND@0, U1BGND.GND@1, U1BGND.GND@10, U1BGND.GND@11, U1BGND.GND@12, U1BGND.GND@2, U1BGND.GND@3, U1BGND.GND@4, U1BGND.GND@5, U1BGND.GND@6, U1BGND.GND@7, U1BGND.GND@8, U1BGND.GND@9, U1BNA.SUSPEND, U4.GND
- net I0: now also U1B0.IO_L36N_GCLK14_0
- net I1: now also U1B0.IO_L36P_GCLK15_0
- net I10: now also U1B0.IO_L2N_0
- net I11: now also U1B0.IO_L2P_0
- net I2: now also U1B0.IO_L35N_GCLK16_0
- net I3: now also U1B0.IO_L35P_GCLK17_0
- net I4: now also U1B0.IO_L34N_GCLK18_0
- net I5: now also U1B0.IO_L34P_GCLK19_0
- net I6: now also U1B0.IO_L4N_0
- net I7: now also U1B0.IO_L4P_0
- net I8: now also U1B0.IO_L3N_0
- net I9: now also U1B0.IO_L3P_0
- net Q0: now also U1B0.IO_L66N_SCP0_0
- net Q1: now also U1B0.IO_L66P_SCP1_0
- net Q10: now also U1B0.IO_L37N_GCLK12_0
- net Q11: now also U1B0.IO_L37P_GCLK13_0
- net Q2: now also U1B0.IO_L65N_SCP2_0
- net Q3: now also U1B0.IO_L65P_SCP3_0
- net Q4: now also U1B0.IO_L64N_SCP4_0
- net Q5: now also U1B0.IO_L64P_SCP5_0
- net Q6: now also U1B0.IO_L63N_SCP6_0
- net Q7: now also U1B0.IO_L63P_SCP7_0
- net Q8: now also U1B0.IO_L62N_VREF_0
- net Q9: now also U1B0.IO_L62P_0
Other:
- note added: "FPGA power supply and config"
- note added: "Output stage and level measurement"

Commit message: MCU added
Parts:
- added C175, C176, C177, C178, C179, C180: 100n, rcl:C-EUC0603
- added IC13: STM32F030C8T, micro-stm_v3:STM32F030C8T
- added JP1: (no value), pinhead:PINHD-1X5
- added JP2: (no value), pinhead:PINHD-1X3
- added Q6: BSS84, transistor-small-signal:BSS84
- added R72, R73: 10k, resistor:R-EU_R0603
- added SV2: (no value), con-ml:ML10
- added TC1: TCXO-NO-VC-CFPT-127, IQD-Frequency-Products:TCXO-NO-VC-CFPT-127
Connections:
- removed net DET_\EN: IC27.ENX, R54.2
- removed net EN_DIREKT: Q1.G
- new net DET_/EN: IC13MCU.PC13, IC27.ENX, R54.2
- new net EN_DIRECT: IC13MCU.PA2, Q1.G
- new net EN_INTREF: Q6.G, R73.1
- new net N$178: IC13MCU.PA10, JP2.1
- new net N$179: IC13MCU.PA9, JP2.3
- new net N$180: IC13MCU.PA14, JP1.2
- new net N$181: C179.1, Q6.D, TC1.VCC
- new net N$182: IC13MCU.PA13, JP1.4
- new net N$183: C178.1, IC13MCU.NRST, JP1.5, R72.1
- new net N$184: IC13MCU.PA8, U1B3.IO_L41P_GCLK27_3
- new net N$185: IC13MCU.PB12, SV2.2
- new net N$186: IC13MCU.PB15, SV2.8
- new net N$187: IC13MCU.PB14, SV2.6
- new net N$188: IC13MCU.PB13, SV2.4
- net +3V3: now also C175.1, C176.1, C177.1, C180.1, IC13MCU.PF7, IC13MCU.VDDA, IC13PWR.VDD@1, IC13PWR.VDD@2, IC13PWR.VDD@3, JP1.1, R72.2, U1B3.VCCO_3@0, U1B3.VCCO_3@1, U1B3.VCCO_3@2
- net +5V: now also SV2.1, SV2.3
- net 10MHZ_REF: now also TC1.OUT
- net 15DB1: now also IC13MCU.OSC_OUT
- net 15DB2: now also IC13MCU.OSC_IN
- net 15DB3: now also IC13MCU.PC15
- net ADF_CE: now also IC13MCU.PA11
- net ADF_LE: now also IC13MCU.PA15
- net ADF_MUX: now also IC13MCU.PA12
- net DBM_CS: now also IC13MCU.PB6
- net DET_SCI1: now also IC13MCU.PB8
- net DET_SCI2: now also IC13MCU.PB9
- net DET_SCI3: now also IC13MCU.PB7
- net DET_SCI4: now also IC13MCU.PC14
- net GND: now also C175.2, C176.2, C177.2, C178.2, C179.2, C180.2, IC13MCU.BOOT0, IC13MCU.PF6, IC13MCU.VSSA, IC13PWR.VSS@1, IC13PWR.VSS@2, JP1.3, JP2.2, SV2.5, SV2.7, SV2.9, TC1.GND
- net PLL_DIG3: now also Q6.S, R73.2
- net SPI_CLK: now also IC13MCU.PB5
- net SPI_MOSI: now also IC13MCU.PB3
Other:
- moved on the sheet: C101, C102, C103, C104, C105, C106, C107, C108, C109, C113, C114, C115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

Commit message: Routing of schematic completed
Parts:
- added C181: 100n, rcl:C-EUC0603
- added C182: 33p, rcl:C-EUC0603
- added R74: 10k, resistor:R-EU_R0603
- added R75, R76: 22, resistor:R-EU_R0603
Connections:
- new net FPGA_CS: IC13MCU.PA6, U1B3.IO_L1P_3
- new net N$189: C181.1, IC13MCU.PA0-WKUP, R74.2
- new net N$190: C182.1, R75.2, U1B3.IO_L43P_GCLK23_3
- new net N$191: IC13MCU.PB4, U1B3.IO_L43N_GCLK22_IRDY2_3
- new net N$192: R76.2, U1B3.IO_L41N_GCLK26_3
- net 10MHZ_REF: now also R76.1
- net ADF_CE: now also IC13MCU.PA5; no longer IC13MCU.PA11
- net ADF_MUX: now also IC13MCU.PA4; no longer IC13MCU.PA12
- net EN_INTREF: now also IC13MCU.PA3
- net ETOUT: now also R74.1
- net GND: now also C181.2, C182.2
- net OFFSET_CS: now also IC13MCU.PB1
- net SPI_CLK: now also R75.1
- net SPI_MOSI: now also U1B3.IO_L44P_GCLK21_3
- net SW1_CTL1: now also U1B3.IO_L83N_VREF_3
- net SW1_CTL2: now also U1B3.IO_L83P_3
- net SW1_CTL3: now also U1B3.IO_L52N_3
- net SW2_CTL1: now also U1B3.IO_L52P_3
- net SW2_CTL2: now also U1B3.IO_L51N_3
- net SW2_CTL3: now also U1B3.IO_L51P_3
- net SYNTH_CE: now also IC13MCU.PA11
- net SYNTH_LE: now also IC13MCU.PB11
- net SYNTH_LOCK_DETECT: now also IC13MCU.PA12
- net SYNTH_MUX: now also IC13MCU.PB10
- net SYNTH_RF_EN: now also IC13MCU.PB2
Other:
- moved on the sheet: JP2, U1B3

Commit message: Via stitching, missing connections, FPGA pins to FFC connector
Parts:
- added C183: 100n, rcl:C-EUC0603
- added LED1, LED2, LED3, LED4, LED5: (no value), led:LEDCHIP-LED0603
- added R77: 10k, resistor:R-EU_R0603
- added R78, R79, R80, R81, R82: 220, resistor:R-EU_R0603
- added X2: FH12-20S-0.5SH, con-hirose:FH12-20S-0.5SH
Connections:
- new net N$157: C183.1, IC13MCU.PA1, R77.2
- new net N$193: U1B1.IO_L42N_GCLK6_TRDY1_1, X2-2.1
- new net N$194: U1B1.IO_L42P_GCLK7_1, X2-3.1
- new net N$195: U1B1.IO_L41N_GCLK8_1, X2-7.1
- new net N$196: U1B1.IO_L41P_GCLK9_IRDY1_1, X2-8.1
- new net N$197: U1B1.IO_L40N_GCLK10_1, X2-9.1
- new net N$198: U1B1.IO_L40P_GCLK11_1, X2-10.1
- new net N$199: U1B1.IO_L34N_1, X2-12.1
- new net N$200: U1B1.IO_L34P_1, X2-13.1
- new net N$201: U1B1.IO_L33N_1, X2-14.1
- new net N$202: U1B1.IO_L32N_1, X2-16.1
- new net N$203: U1B1.IO_L32P_1, X2-17.1
- new net N$204: U1B1.IO_L1N_VREF_1, X2-19.1
- new net N$205: U1B1.IO_L1P_1, X2-20.1
- new net N$206: LED1.C, R78.2
- new net N$207: LED2.C, R79.2
- new net N$208: LED3.C, R80.2
- new net N$209: LED4.C, R81.2
- new net N$210: LED5.C, R82.2
- new net N$211: LED1.A, U1B1.IO_L74N_DOUT_BUSY_1
- new net N$212: LED2.A, U1B1.IO_L74P_AWAKE_1
- new net N$213: LED3.A, U1B1.IO_L47N_1
- new net N$214: LED4.A, U1B1.IO_L47P_1
- new net N$215: LED5.A, U1B1.IO_L46N_1
- new net RMSOUT: C155.1, IC27.VSET, R59.1, R60.2, R61.1, R77.1
- net +3V3: now also U1B1.VCCO_1@0, U1B1.VCCO_1@1, U1B1.VCCO_1@2, X2-1.1, X2-18.1, X2-5.1
- net DORI: now also U1B3.IO_L50N_3
- net GND: now also C183.2, IC6.PD, R78.1, R79.1, R80.1, R81.1, R82.1, X2-11.1, X2-6.1
- net MIX_EN: now also IC13MCU.PB0
- net N$162: now also U1B1.IO_L33P_1, X2-15.1; no longer C155.1, IC27.VSET, R59.1, R60.2, R61.1
- net SELIQ: now also U1B3.IO_L50P_3
- net VCCINT: now also X2-4.1
