File: Hardware/RFBoard.brd (EAGLE design)
At the start: 100 x 100 mm, 388 parts, among them IC1 HMC1097, IC10 NCP702-1.8, IC11 TPS42951, IC12 MCP4812, IC13 STM32F030C8T, IC14 LT5560, IC15 ADF4360, IC16 HMC284, IC17 HMC284, IC18 NCP702-3.3, IC19 NCP702-3.3, IC2 MAX2871, IC20 LT1395, IC21 MAADSS0008, IC22 MAADSS0008, IC23 MAADSS0008, IC24 RFSA2033, IC25 MMG3H21NT1, IC26 MMG3H21NT1, IC27 HMC1021, IC28 MCP4812, IC29 NCP702-3.3, IC3 AP2114HA-3.3, IC31 QPC6064, IC32 QPC6064, IC4 NCP702-3.3, IC5 NCP702-3.3, IC6 MAX5873, IC7 NCP702-1.8, IC8 NCP702-3.3, IC9 NCP702-3.3, Q1 BSS123, Q2 BSS123, Q3 BSS123, Q4 BSS123, Q5 BSS123, Q6 BSS84, U1 6SLX9TQG144, U4 W25Q16BVSN, X1 out, X2 FH12-20S-0.5SH

Commit message: PCB finished
Parts:
- added C184: 100n, rcl:C0603
- added J1: U.FL-R-SMT, connector:U.FL_SMT
Connections:
- new net N$178: C184.2, J1.SIG
- net 10MHZ_REF: now also C184.1
- net GND: now also J1.GND1, J1.GND2
Routing:
- net GND: track 2267.6 -> 2280.9 mm, vias 996 -> 1001
- net N$178: track 0.00 -> 2.55 mm
- net 10MHZ_REF: track 21.6 -> 23.2 mm
Other:
- board text added: "ExtRef"
Changed lines of the file:
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@@
 <layer number="54" name="bPadExt" color="1" fill="1" visible="no" active="no"/>
 <layer number="56" name="wert" color="7" fill="1" visible="no" active="yes"/>
+<layer number="57" name="tCAD" color="7" fill="1" visible="no" active="no"/>
 <layer number="88" name="SimResults" color="9" fill="1" visible="no" active="no"/>
 <layer number="89" name="SimProbes" color="9" fill="1" visible="no" active="no"/>
@@
 <layer number="99" name="SpiceOrder" color="5" fill="1" visible="no" active="no"/>
 <layer number="100" name="Muster" color="7" fill="1" visible="no" active="no"/>
+<layer number="101" name="Patch_Top" color="12" fill="4" visible="no" active="yes"/>
+<layer number="102" name="Vscore" color="7" fill="1" visible="no" active="yes"/>
+<layer number="103" name="tMap" color="7" fill="1" visible="no" active="yes"/>
+<layer number="104" name="Name" color="16" fill="1" visible="no" active="yes"/>
+<layer number="105" name="tPlate" color="7" fill="1" visible="no" active="yes"/>
+<layer number="106" name="bPlate" color="7" fill="1" visible="no" active="yes"/>
+<layer number="107" name="Crop" color="2" fill="1" visible="no" active="yes"/>
+<layer number="108" name="fp8" color="7" fill="1" visible="no" active="yes"/>
+<layer number="109" name="fp9" color="7" fill="1" visible="no" active="yes"/>
+<layer number="110" name="fp0" color="7" fill="1" visible="no" active="yes"/>
+<layer number="111" name="LPC17xx" color="7" fill="1" visible="no" active="yes"/>
+<layer number="112" name="tSilk" color="7" fill="1" visible="no" active="yes"/>
+<layer number="113" name="IDFDebug" color="7" fill="1" visible="no" active="yes"/>
+<layer number="116" name="Patch_BOT" color="9" fill="4" visible="no" active="yes"/>
+<layer number="121" name="_tsilk" color="7" fill="1" visible="no" active="yes"/>
+<layer number="122" name="_bsilk" color="7" fill="1" visible="no" active="yes"/>
+<layer number="123" name="tTestmark" color="7" fill="1" visible="no" active="yes"/>
+<layer number="124" name="bTestmark" color="7" fill="1" visible="no" active="yes"/>
+<layer number="125" name="_tNames" color="7" fill="1" visible="no" active="yes"/>
+<layer number="126" name="_bNames" color="7" fill="1" visible="no" active="yes"/>
+<layer number="127" name="_tValues" color="7" fill="1" visible="no" active="yes"/>
+<layer number="128" name="_bValues" color="7" fill="1" visible="no" active="yes"/>
+<layer number="131" name="tAdjust" color="7" fill="1" visible="no" active="yes"/>
+<layer number="132" name="bAdjust" color="7" fill="1" visible="no" active="yes"/>
+<layer number="144" name="Drill_legend" color="7" fill="1" visible="no" active="yes"/>
+<layer number="150" name="Notes" color="7" fill="1" visible="no" active="yes"/>
+<layer number="151" name="HeatSink" color="7" fill="1" visible="no" active="yes"/>
+<layer number="152" name="_bDocu" color="7" fill="1" visible="no" active="yes"/>
+<layer number="153" name="FabDoc1" color="7" fill="1" visible="no" active="yes"/>
+<layer number="154" name="FabDoc2" color="7" fill="1" visible="no" active="yes"/>
+<layer number="155" name="FabDoc3" color="7" fill="1" visible="no" active="yes"/>
+<layer number="199" name="Contour" color="7" fill="1" visible="no" active="yes"/>
+<layer number="200" name="200bmp" color="1" fill="10" visible="no" active="yes"/>
+<layer number="201" name="201bmp" color="1" fill="10" visible="no" active="yes"/>
+<layer number="202" name="202bmp" color="3" fill="10" visible="no" active="yes"/>
+<layer number="203" name="203bmp" color="4" fill="10" visible="no" active="yes"/>
+<layer number="204" name="204bmp" color="5" fill="10" visible="no" active="yes"/>
+<layer number="205" name="205bmp" color="6" fill="10" visible="no" active="yes"/>
+<layer number="206" name="206bmp" color="7" fill="10" visible="no" active="yes"/>
+<layer number="207" name="207bmp" color="8" fill="10" visible="no" active="yes"/>
+<layer number="208" name="208bmp" color="9" fill="10" visible="no" active="yes"/>
+<layer number="209" name="209bmp" color="7" fill="1" visible="no" active="yes"/>
+<layer number="210" name="210bmp" color="7" fill="1" visible="no" active="yes"/>
+<layer number="211" name="211bmp" color="7" fill="1" visible="no" active="yes"/>
+<layer number="212" name="212bmp" color="7" fill="1" visible="no" active="yes"/>
+<layer number="213" name="213bmp" color="7" fill="1" visible="no" active="yes"/>
+<layer number="214" name="214bmp" color="7" fill="1" visible="no" active="yes"/>
+<layer number="215" name="215bmp" color="7" fill="1" visible="no" active="yes"/>
+<layer number="216" name="216bmp" color="7" fill="1" visible="no" active="yes"/>
+<layer number="217" name="217bmp" color="18" fill="1" visible="no" active="no"/>
+<layer number="218" name="218bmp" color="19" fill="1" visible="no" active="no"/>
+<layer number="219" name="219bmp" color="20" fill="1" visible="no" active="no"/>
+<layer number="220" name="220bmp" color="21" fill="1" visible="no" active="no"/>
+<layer number="221" name="221bmp" color="22" fill="1" visible="no" active="no"/>
+<layer number="222" name="222bmp" color="23" fill="1" visible="no" active="no"/>
+<layer number="223" name="223bmp" color="24" fill="1" visible="no" active="no"/>
+<layer number="224" name="224bmp" color="25" fill="1" visible="no" active="no"/>
+<layer number="248" name="Housing" color="7" fill="1" visible="no" active="yes"/>
+<layer number="249" name="Edge" color="7" fill="1" visible="no" active="yes"/>
 <layer number="250" name="Descript" color="3" fill="1" visible="no" active="no"/>
 <layer number="251" name="SMDround" color="12" fill="11" visible="no" active="no"/>
+<layer number="254" name="cooling" color="7" fill="1" visible="no" active="yes"/>
 </layers>
 <board>
@@
 <text x="58.5" y="88" size="1.778" layer="22" font="vector" rot="MR0">Rev. A</text>
 <text x="85" y="86" size="1.4224" layer="22" font="vector" rot="MR0">github.com/jankae/Signalgenerator</text>
+<text x="52.7" y="51.4" size="1.016" layer="22" font="vector" rot="MR270">ExtRef</text>
 </plain>
 <attributes>
@@
 <attribute name="VALUE" x="61.405" y="2.635" size="1.27" layer="28" rot="MR270"/>
 </element>
+<element name="J1" library="connector" package="U.FL_SMT" value="U.FL-R-SMT" x="49.5" y="50" smashed="yes" rot="MR90">
+<attribute name="DIGIKEY" value="H122041-ND" x="49.5" y="50" size="1.778" layer="28" rot="MR90" display="off"/>
+<attribute name="MANUFACTURER" value="Hirose" x="49.5" y="50" size="1.778" layer="28" rot="MR90" display="off"/>
+<attribute name="MPN" value="U.FL-R-SMT-1(01)" x="49.5" y="50" size="1.778" layer="28" rot="MR90" display="off"/>
+<attribute name="NAME" x="47.094" y="50.1" size="0.8128" layer="26" font="vector" ratio="12" rot="MR270" align="bottom-center"/>
+</element>
+<element name="C184" library="rcl" package="C0603" value="100n" x="47" y="53" smashed="yes" rot="MR270">
+<attribute name="NAME" x="46.165" y="54.335" size="0.8128" layer="26" font="vector" rot="MR270"/>
+<attribute name="VALUE" x="48.905" y="53.635" size="1.27" layer="28" rot="MR270"/>
+</element>
 </elements>
 <signals>
@@
 <wire x1="74.5" y1="45.5" x2="65.2" y2="45.5" width="3" layer="16"/>
 <wire x1="65.2" y1="45.5" x2="58.7" y2="45.5" width="3" layer="16"/>
-<wire x1="58.7" y1="45.5" x2="44.5" y2="45.5" width="3" layer="16"/>
+<wire x1="58.7" y1="45.5" x2="49.4" y2="45.5" width="3" layer="16"/>
+<wire x1="49.4" y1="45.5" x2="44.5" y2="45.5" width="3" layer="16"/>
 <wire x1="44.5" y1="45.5" x2="43.5" y2="45.5" width="3" layer="16"/>
 <wire x1="43.5" y1="45.5" x2="42.5" y2="45.5" width="3" layer="16"/>
@@
 <wire x1="57.55" y1="7.9" x2="56.5" y2="6.85" width="0.3" layer="16"/>
 <wire x1="56.5" y1="6.85" x2="56.5" y2="2.85" width="0.3" layer="16"/>
+<contactref element="J1" pad="GND1"/>
+<contactref element="J1" pad="GND2"/>
+<wire x1="49.5" y1="48.525" x2="49.5" y2="45.6" width="0.6" layer="16"/>
+<wire x1="49.5" y1="45.6" x2="49.4" y2="45.5" width="0.6" layer="16"/>
+<wire x1="49.5" y1="51.475" x2="49.5" y2="53.35" width="0.6" layer="16"/>
+<wire x1="49.5" y1="53.35" x2="50.3" y2="54.15" width="0.6" layer="16"/>
+<via x="49.5" y="47.6" extent="1-16" drill="0.25"/>
+<via x="51.3" y="48.5" extent="1-16" drill="0.25"/>
+<via x="51.3" y="51.5" extent="1-16" drill="0.25"/>
+<via x="48.7" y="52.5" extent="1-16" drill="0.25"/>
+<via x="47.8" y="48.6" extent="1-16" drill="0.25"/>
+<wire x1="47.8" y1="48.6" x2="49.425" y2="48.6" width="0.6" layer="16"/>
+<wire x1="49.425" y1="48.6" x2="49.5" y2="48.525" width="0.6" layer="16"/>
+<wire x1="51.3" y1="48.5" x2="49.525" y2="48.5" width="0.6" layer="16"/>
+<wire x1="49.525" y1="48.5" x2="49.425" y2="48.6" width="0.6" layer="16"/>
+<wire x1="51.3" y1="51.5" x2="49.525" y2="51.5" width="0.6" layer="16"/>
+<wire x1="49.525" y1="51.5" x2="49.5" y2="51.475" width="0.6" layer="16"/>
+<wire x1="48.7" y1="52.5" x2="48.7" y2="51.5" width="0.6" layer="16"/>
+<wire x1="48.7" y1="51.5" x2="48.725" y2="51.475" width="0.6" layer="16"/>
+<wire x1="48.725" y1="51.475" x2="49.5" y2="51.475" width="0.6" layer="16"/>
 <wire x1="83.993" y1="28.4" x2="83.993" y2="27.9" width="0" layer="19" extent="1-1"/>
 </signal>
@@
 <wire x1="47" y1="52.85" x2="47" y2="54.85" width="0.3" layer="1"/>
 <wire x1="47" y1="54.85" x2="46.9" y2="54.95" width="0.3" layer="1"/>
+<contactref element="C184" pad="1"/>
+<wire x1="47" y1="53.85" x2="47" y2="54" width="0.3" layer="16"/>
+<wire x1="47" y1="54" x2="46" y2="55" width="0.3" layer="16"/>
 </signal>
 <signal name="N$12">
@@
 <wire x1="60.8" y1="27.5" x2="60.55" y2="27.75" width="0.3" layer="1"/>
 </signal>
+<signal name="N$178">
+<contactref element="C184" pad="2"/>
+<contactref element="J1" pad="SIG"/>
+<wire x1="47.975" y1="50" x2="47" y2="50.975" width="0.3" layer="16"/>
+<wire x1="47" y1="50.975" x2="47" y2="52.15" width="0.3" layer="16"/>
+</signal>
 </signals>

Commit message: PLL loop filter values changed
Parts:
- C102, C5: value 820p -> 10n
- C103: value 100n -> 330p
- C104: value 820p -> 220p
- C4: value 12n -> 10n
- R1: value 250 -> 330
- R15: value 73k2 -> 15k
- R2: value 0 -> 270
- R27: value 250 -> 15k
- R29: value 120 -> 6k8
- R3: value 120 -> 1k
- R66: value 22k1 -> 11k
Changed lines of the file:
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@@
 <attribute name="VALUE" x="25.095" y="58.935" size="1.27" layer="27" rot="R270"/>
 </element>
-<element name="C102" library="rcl" package="C0603" value="820p" x="34.8" y="55.3" smashed="yes" rot="R90">
+<element name="C102" library="rcl" package="C0603" value="10n" x="34.8" y="55.3" smashed="yes" rot="R90">
 <attribute name="NAME" x="37.165" y="54.165" size="0.8128" layer="25" font="vector" rot="R90"/>
 <attribute name="VALUE" x="36.705" y="54.665" size="1.27" layer="27" rot="R90"/>
 </element>
-<element name="C103" library="rcl" package="C0603" value="100n" x="38.4" y="58.6" smashed="yes" rot="R270">
+<element name="C103" library="rcl" package="C0603" value="330p" x="38.4" y="58.6" smashed="yes" rot="R270">
 <attribute name="NAME" x="40.035" y="60.735" size="0.8128" layer="25" font="vector" rot="R270"/>
 <attribute name="VALUE" x="36.495" y="59.235" size="1.27" layer="27" rot="R270"/>
 </element>
-<element name="C104" library="rcl" package="C0603" value="820p" x="34.8" y="58.6" smashed="yes" rot="R270">
+<element name="C104" library="rcl" package="C0603" value="220p" x="34.8" y="58.6" smashed="yes" rot="R270">
 <attribute name="NAME" x="34.465" y="60.135" size="0.8128" layer="25" font="vector"/>
 <attribute name="VALUE" x="32.895" y="59.235" size="1.27" layer="27" rot="R270"/>
@@
 <attribute name="VALUE" x="95.865" y="25.495" size="1.27" layer="27"/>
 </element>
-<element name="C4" library="rcl" package="C0603" value="12n" x="63.01" y="48.51" smashed="yes">
+<element name="C4" library="rcl" package="C0603" value="10n" x="63.01" y="48.51" smashed="yes">
 <attribute name="NAME" x="62.675" y="49.345" size="0.8128" layer="25" font="vector"/>
 <attribute name="VALUE" x="62.375" y="46.605" size="1.27" layer="27"/>
@@
 <attribute name="VALUE" x="84.465" y="40.095" size="1.27" layer="27"/>
 </element>
-<element name="C5" library="rcl" package="C0603" value="820p" x="61.8" y="58.9" smashed="yes" rot="MR270">
+<element name="C5" library="rcl" package="C0603" value="10n" x="61.8" y="58.9" smashed="yes" rot="MR270">
 <attribute name="NAME" x="60.765" y="59.435" size="1.016" layer="26" font="vector" rot="MR270"/>
 <attribute name="VALUE" x="63.705" y="59.535" size="1.27" layer="28" rot="MR270"/>
@@
 <attribute name="VALUE" x="3.595" y="48.175" size="1.27" layer="28" rot="MR180"/>
 </element>
-<element name="R1" library="resistor" package="R0603" value="250" x="61.8" y="54.5" smashed="yes" rot="MR90">
+<element name="R1" library="resistor" package="R0603" value="330" x="61.8" y="54.5" smashed="yes" rot="MR90">
 <attribute name="NAME" x="62.435" y="56.235" size="1.016" layer="26" font="vector" rot="MR0"/>
 <attribute name="VALUE" x="59.895" y="53.865" size="1.27" layer="28" rot="MR90"/>
@@
 <attribute name="VALUE" x="88.205" y="31.235" size="1.27" layer="28" rot="MR270"/>
 </element>
-<element name="R2" library="resistor" package="R0603" value="0" x="55.4" y="48.5" smashed="yes" rot="R180">
+<element name="R2" library="resistor" package="R0603" value="270" x="55.4" y="48.5" smashed="yes" rot="R180">
 <attribute name="NAME" x="56.135" y="50.165" size="0.8128" layer="25" font="vector" rot="R180"/>
 <attribute name="VALUE" x="56.035" y="50.405" size="1.27" layer="27" rot="R180"/>
@@
 <attribute name="VALUE" x="91.135" y="34.995" size="1.27" layer="28" rot="MR0"/>
 </element>
-<element name="R27" library="resistor" package="R0603" value="250" x="36.6" y="58.6" smashed="yes" rot="R270">
+<element name="R27" library="resistor" package="R0603" value="15k" x="36.6" y="58.6" smashed="yes" rot="R270">
 <attribute name="NAME" x="39.035" y="60.335" size="0.8128" layer="25" font="vector" rot="R270"/>
 <attribute name="VALUE" x="34.695" y="59.235" size="1.27" layer="27" rot="R270"/>
@@
 <attribute name="VALUE" x="91.135" y="36.695" size="1.27" layer="28" rot="MR0"/>
 </element>
-<element name="R29" library="resistor" package="R0603" value="120" x="38.4" y="55.3" smashed="yes" rot="R270">
+<element name="R29" library="resistor" package="R0603" value="6k8" x="38.4" y="55.3" smashed="yes" rot="R270">
 <attribute name="NAME" x="39.335" y="56.335" size="0.8128" layer="25" font="vector" rot="R270"/>
 <attribute name="VALUE" x="36.495" y="55.935" size="1.27" layer="27" rot="R270"/>
 </element>
-<element name="R3" library="resistor" package="R0603" value="120" x="51.8" y="48.5" smashed="yes" rot="R180">
+<element name="R3" library="resistor" package="R0603" value="1k" x="51.8" y="48.5" smashed="yes" rot="R180">
 <attribute name="NAME" x="50.035" y="48.865" size="0.8128" layer="25" font="vector" rot="R180"/>
 <attribute name="VALUE" x="52.435" y="50.405" size="1.27" layer="27" rot="R180"/>
@@
 <attribute name="VALUE" x="43.54" y="10.43" size="1.27" layer="27" rot="R90"/>
 </element>
-<element name="R15" library="resistor" package="R0603" value="73k2" x="40.5" y="2.7" smashed="yes" rot="R180">
+<element name="R15" library="resistor" package="R0603" value="15k" x="40.5" y="2.7" smashed="yes" rot="R180">
 <attribute name="NAME" x="41.535" y="1.765" size="0.8128" layer="25" font="vector" rot="R180"/>
 <attribute name="VALUE" x="41.135" y="4.605" size="1.27" layer="27" rot="R180"/>
 </element>
-<element name="R66" library="resistor" package="R0603" value="22k1" x="35.5" y="3.2" smashed="yes" rot="R270">
+<element name="R66" library="resistor" package="R0603" value="11k" x="35.5" y="3.2" smashed="yes" rot="R270">
 <attribute name="NAME" x="34.865" y="0.135" size="0.8128" layer="25" font="vector"/>
 <attribute name="VALUE" x="33.595" y="3.835" size="1.27" layer="27" rot="R270"/>
