File: Hardware/RFBoard.brd (EAGLE design)
At the start: 100 x 100 mm, 390 parts, among them IC1 HMC1097, IC10 NCP702-1.8, IC11 TPS42951, IC12 MCP4812, IC13 STM32F030C8T, IC14 LT5560, IC15 ADF4360, IC16 HMC284, IC17 HMC284, IC18 NCP702-3.3, IC19 NCP702-3.3, IC2 MAX2871, IC20 LT1395, IC21 MAADSS0008, IC22 MAADSS0008, IC23 MAADSS0008, IC24 RFSA2033, IC25 MMG3H21NT1, IC26 MMG3H21NT1, IC27 HMC1021, IC28 MCP4812, IC29 NCP702-3.3, IC3 AP2114HA-3.3, IC31 QPC6064, IC32 QPC6064, IC4 NCP702-3.3, IC5 NCP702-3.3, IC6 MAX5873, IC7 NCP702-1.8, IC8 NCP702-3.3, IC9 NCP702-3.3, J1 U.FL-R-SMT, Q1 BSS123, Q2 BSS123, Q3 BSS123, Q4 BSS123, Q5 BSS123, Q6 BSS84, U1 6SLX9TQG144, U4 W25Q16BVSN, X1 out, X2 FH12-20S-0.5SH

Commit message: Value changes amplitude control feedback loop
Parts:
- C153, C154, C155: value 1u -> DNP
- R60: value DNP -> 1u
Changed lines of the file:
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@@
 <attribute name="VALUE" x="19.095" y="59.135" size="1.27" layer="27" rot="R270"/>
 </element>
-<element name="C153" library="rcl" package="C0603" value="1u" x="13" y="51" smashed="yes" rot="R270">
+<element name="C153" library="rcl" package="C0603" value="DNP" x="13" y="51" smashed="yes" rot="R270">
 <attribute name="NAME" x="12.265" y="49.265" size="0.8128" layer="25" font="vector" rot="R90"/>
 <attribute name="VALUE" x="11.095" y="51.635" size="1.27" layer="27" rot="R270"/>
 </element>
-<element name="C154" library="rcl" package="C0603" value="1u" x="13" y="58.5" smashed="yes" rot="R90">
+<element name="C154" library="rcl" package="C0603" value="DNP" x="13" y="58.5" smashed="yes" rot="R90">
 <attribute name="NAME" x="12.265" y="58.365" size="0.8128" layer="25" font="vector" rot="R90"/>
 <attribute name="VALUE" x="14.905" y="57.865" size="1.27" layer="27" rot="R90"/>
 </element>
-<element name="C155" library="rcl" package="C0603" value="1u" x="20" y="50.3" smashed="yes">
+<element name="C155" library="rcl" package="C0603" value="DNP" x="20" y="50.3" smashed="yes">
 <attribute name="NAME" x="20.165" y="51.135" size="0.8128" layer="25" font="vector"/>
 <attribute name="VALUE" x="19.365" y="48.395" size="1.27" layer="27"/>
@@
 <attribute name="VALUE" x="19.365" y="46.695" size="1.27" layer="27"/>
 </element>
-<element name="R60" library="resistor" package="R0603" value="DNP" x="16.97" y="48.61" smashed="yes">
+<element name="R60" library="resistor" package="R0603" value="1u" x="16.97" y="48.61" smashed="yes">
 <attribute name="NAME" x="17.435" y="47.045" size="0.8128" layer="25" font="vector"/>
 <attribute name="VALUE" x="16.335" y="46.705" size="1.27" layer="27"/>

Commit message: External modulation input usable as modulation source
Parts:
- C4: value 10n -> 2n
- C5: value 10n -> 180p
- C6: value 100n -> 33n
- R1: value 330 -> 1k
- R2: value 270 -> 100
- R3: value 1k -> 120
Changed lines of the file:
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@@
 <attribute name="VALUE" x="95.865" y="25.495" size="1.27" layer="27"/>
 </element>
-<element name="C4" library="rcl" package="C0603" value="10n" x="63.01" y="48.51" smashed="yes">
+<element name="C4" library="rcl" package="C0603" value="2n" x="63.01" y="48.51" smashed="yes">
 <attribute name="NAME" x="62.675" y="49.345" size="0.8128" layer="25" font="vector"/>
 <attribute name="VALUE" x="62.375" y="46.605" size="1.27" layer="27"/>
@@
 <attribute name="VALUE" x="84.465" y="40.095" size="1.27" layer="27"/>
 </element>
-<element name="C5" library="rcl" package="C0603" value="10n" x="61.8" y="58.9" smashed="yes" rot="MR270">
+<element name="C5" library="rcl" package="C0603" value="180p" x="61.8" y="58.9" smashed="yes" rot="MR270">
 <attribute name="NAME" x="60.765" y="59.435" size="1.016" layer="26" font="vector" rot="MR270"/>
 <attribute name="VALUE" x="63.705" y="59.535" size="1.27" layer="28" rot="MR270"/>
@@
 <attribute name="VALUE" x="90.865" y="67.595" size="1.27" layer="27"/>
 </element>
-<element name="C6" library="rcl" package="C0603" value="100n" x="58.6" y="48.5" smashed="yes" rot="R180">
+<element name="C6" library="rcl" package="C0603" value="33n" x="58.6" y="48.5" smashed="yes" rot="R180">
 <attribute name="NAME" x="58.935" y="50.065" size="0.8128" layer="25" font="vector" rot="R180"/>
 <attribute name="VALUE" x="59.235" y="50.405" size="1.27" layer="27" rot="R180"/>
@@
 <attribute name="VALUE" x="3.595" y="48.175" size="1.27" layer="28" rot="MR180"/>
 </element>
-<element name="R1" library="resistor" package="R0603" value="330" x="61.8" y="54.5" smashed="yes" rot="MR90">
+<element name="R1" library="resistor" package="R0603" value="1k" x="61.8" y="54.5" smashed="yes" rot="MR90">
 <attribute name="NAME" x="62.435" y="56.235" size="1.016" layer="26" font="vector" rot="MR0"/>
 <attribute name="VALUE" x="59.895" y="53.865" size="1.27" layer="28" rot="MR90"/>
@@
 <attribute name="VALUE" x="88.205" y="31.235" size="1.27" layer="28" rot="MR270"/>
 </element>
-<element name="R2" library="resistor" package="R0603" value="270" x="55.4" y="48.5" smashed="yes" rot="R180">
+<element name="R2" library="resistor" package="R0603" value="100" x="55.4" y="48.5" smashed="yes" rot="R180">
 <attribute name="NAME" x="56.135" y="50.165" size="0.8128" layer="25" font="vector" rot="R180"/>
 <attribute name="VALUE" x="56.035" y="50.405" size="1.27" layer="27" rot="R180"/>
@@
 <attribute name="VALUE" x="36.495" y="55.935" size="1.27" layer="27" rot="R270"/>
 </element>
-<element name="R3" library="resistor" package="R0603" value="1k" x="51.8" y="48.5" smashed="yes" rot="R180">
+<element name="R3" library="resistor" package="R0603" value="120" x="51.8" y="48.5" smashed="yes" rot="R180">
 <attribute name="NAME" x="50.035" y="48.865" size="0.8128" layer="25" font="vector" rot="R180"/>
 <attribute name="VALUE" x="52.435" y="50.405" size="1.27" layer="27" rot="R180"/>
