File: Hardware/IQInput.brd (EAGLE design)
At the start: 50 x 50 mm, 100 parts, among them IC1 TPS60403, IC2 LT1819, IC3 AD8132, IC4 AD8132, IC5 MAX19515, IC6 PCA9555BS, K1 FTR-B4G, K2 FTR-B4G, K3 FTR-B4G, K4 FTR-B4G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

Commit message: Part values corrected
Parts:
- C10, C3, C4, C9: value DNP -> 33p
- R11, R25: value 750k -> 750k||18p
- R12, R26: value 190k -> 190k||68p
- R13, R27: value 60k -> 60k||220p
- R14, R28: value 10k -> 1k
Changed lines of the file:
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@@
 <attribute name="VALUE" x="26.135" y="17.405" size="1.27" layer="27" rot="R180"/>
 </element>
-<element name="C10" library="rcl" package="C0603" value="DNP" x="36" y="21" smashed="yes" rot="R270">
+<element name="C10" library="rcl" package="C0603" value="33p" x="36" y="21" smashed="yes" rot="R270">
 <attribute name="NAME" x="45.5" y="9.4" size="1.016" layer="25" font="vector" rot="R270"/>
 <attribute name="VALUE" x="34.095" y="21.635" size="1.27" layer="27" rot="R270"/>
@@
 <attribute name="VALUE" x="27.905" y="7.365" size="1.27" layer="27" rot="R90"/>
 </element>
-<element name="C3" library="rcl" package="C0603" value="DNP" x="34" y="21" smashed="yes" rot="R270">
+<element name="C3" library="rcl" package="C0603" value="33p" x="34" y="21" smashed="yes" rot="R270">
 <attribute name="NAME" x="42.8" y="9.2" size="1.016" layer="25" font="vector" rot="R270"/>
 <attribute name="VALUE" x="32.095" y="21.635" size="1.27" layer="27" rot="R270"/>
 </element>
-<element name="C4" library="rcl" package="C0603" value="DNP" x="24" y="21" smashed="yes" rot="R270">
+<element name="C4" library="rcl" package="C0603" value="33p" x="24" y="21" smashed="yes" rot="R270">
 <attribute name="NAME" x="22.135" y="21.435" size="1.016" layer="25" font="vector" rot="R270"/>
 <attribute name="VALUE" x="22.095" y="21.635" size="1.27" layer="27" rot="R270"/>
@@
 <attribute name="VALUE" x="41.685" y="18.985" size="1.27" layer="27" rot="R180"/>
 </element>
-<element name="C9" library="rcl" package="C0603" value="DNP" x="46" y="21" smashed="yes" rot="R270">
+<element name="C9" library="rcl" package="C0603" value="33p" x="46" y="21" smashed="yes" rot="R270">
 <attribute name="NAME" x="48.235" y="21.735" size="1.016" layer="25" font="vector" rot="R270"/>
 <attribute name="VALUE" x="44.095" y="21.635" size="1.27" layer="27" rot="R270"/>
@@
 <attribute name="VALUE" x="15.96" y="41.67" size="1.27" layer="27" rot="R270"/>
 </element>
-<element name="R11" library="rcl" package="R0603" value="750k" x="20.6" y="36.3" smashed="yes" rot="R270">
+<element name="R11" library="rcl" package="R0603" value="750k||18p" x="20.6" y="36.3" smashed="yes" rot="R270">
 <attribute name="NAME" x="20.065" y="37.935" size="1.016" layer="25" font="vector"/>
 <attribute name="VALUE" x="18.695" y="36.935" size="1.27" layer="27" rot="R270"/>
 </element>
-<element name="R12" library="rcl" package="R0603" value="190k" x="20.6" y="43.8" smashed="yes" rot="R270">
+<element name="R12" library="rcl" package="R0603" value="190k||68p" x="20.6" y="43.8" smashed="yes" rot="R270">
 <attribute name="NAME" x="18.835" y="46.235" size="1.016" layer="25" font="vector" rot="R270"/>
 <attribute name="VALUE" x="18.695" y="44.435" size="1.27" layer="27" rot="R270"/>
 </element>
-<element name="R13" library="rcl" package="R0603" value="60k" x="20.6" y="47.5" smashed="yes" rot="R270">
+<element name="R13" library="rcl" package="R0603" value="60k||220p" x="20.6" y="47.5" smashed="yes" rot="R270">
 <attribute name="NAME" x="17.735" y="48.735" size="1.016" layer="25" font="vector" rot="R270"/>
 <attribute name="VALUE" x="18.695" y="48.135" size="1.27" layer="27" rot="R270"/>
 </element>
-<element name="R14" library="rcl" package="R0603" value="10k" x="32.2" y="32.4" smashed="yes">
+<element name="R14" library="rcl" package="R0603" value="1k" x="32.2" y="32.4" smashed="yes">
 <attribute name="NAME" x="33.665" y="31.235" size="0.8128" layer="25" font="vector"/>
 <attribute name="VALUE" x="31.565" y="30.495" size="1.27" layer="27"/>
@@
 <attribute name="VALUE" x="18.54" y="15.23" size="1.27" layer="27" rot="R90"/>
 </element>
-<element name="R25" library="rcl" package="R0603" value="750k" x="32" y="37" smashed="yes" rot="R270">
+<element name="R25" library="rcl" package="R0603" value="750k||18p" x="32" y="37" smashed="yes" rot="R270">
 <attribute name="NAME" x="31.435" y="40.535" size="0.8128" layer="25" font="vector" rot="R270"/>
 <attribute name="VALUE" x="30.095" y="37.635" size="1.27" layer="27" rot="R270"/>
 </element>
-<element name="R26" library="rcl" package="R0603" value="190k" x="34.3" y="40" smashed="yes" rot="R180">
+<element name="R26" library="rcl" package="R0603" value="190k||68p" x="34.3" y="40" smashed="yes" rot="R180">
 <attribute name="NAME" x="37.135" y="41.565" size="0.8128" layer="25" font="vector" rot="R180"/>
 <attribute name="VALUE" x="34.935" y="41.905" size="1.27" layer="27" rot="R180"/>
 </element>
-<element name="R27" library="rcl" package="R0603" value="60k" x="40" y="41" smashed="yes" rot="R270">
+<element name="R27" library="rcl" package="R0603" value="60k||220p" x="40" y="41" smashed="yes" rot="R270">
 <attribute name="NAME" x="38.435" y="42.035" size="0.8128" layer="25" font="vector" rot="R270"/>
 <attribute name="VALUE" x="38.095" y="41.635" size="1.27" layer="27" rot="R270"/>
 </element>
-<element name="R28" library="rcl" package="R0603" value="10k" x="32.2" y="34.4" smashed="yes">
+<element name="R28" library="rcl" package="R0603" value="1k" x="32.2" y="34.4" smashed="yes">
 <attribute name="NAME" x="33.7" y="35.2" size="0.8128" layer="25" font="vector" rot="R90"/>
 <attribute name="VALUE" x="31.565" y="32.495" size="1.27" layer="27"/>
