File: Hardware/IQInput.sch (EAGLE design)
At the start: 97 parts, among them IC1 TPS60403, IC2 LT1819, IC3 AD8132, IC4 AD8132, IC5 MAX19515, IC6 PCA9555BS, K1 FTR-B4G, K2 FTR-B4G, K3 FTR-B4G, K4 FTR-B4G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

Commit message: Added value to input protection resistor
Parts:
- R14, R28: value (none) -> 10k
Changed lines of the file:
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@@
 <part name="K3" library="relay" deviceset="FTR-B4" device="G"/>
 <part name="K4" library="relay" deviceset="FTR-B4" device="G"/>
-<part name="R14" library="rcl" deviceset="R-EU_" device="R0603"/>
+<part name="R14" library="rcl" deviceset="R-EU_" device="R0603" value="10k"/>
 <part name="D3" library="diode" deviceset="BAV199" device=""/>
 <part name="D1" library="diode" deviceset="BAV199" device=""/>
@@
 <part name="R27" library="rcl" deviceset="R-EU_" device="R0603" value="60k"/>
 <part name="GND12" library="supply1" deviceset="GND" device=""/>
-<part name="R28" library="rcl" deviceset="R-EU_" device="R0603"/>
+<part name="R28" library="rcl" deviceset="R-EU_" device="R0603" value="10k"/>
 <part name="D2" library="diode" deviceset="BAV199" device=""/>
 <part name="D4" library="diode" deviceset="BAV199" device=""/>

Commit message: Specified values
Parts:
- C1, C7: value (none) -> 100n
- C10, C3, C4, C9: value (none) -> DNP
- C2, C8: value (none) -> 100p
- L1, L2: value (none) -> Ferrite
- R1, R15, R16, R2: value (none) -> 49R9
- R17, R18, R19, R20, R3, R4, R5, R6: value (none) -> 470
Changed lines of the file:
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@@
 <part name="P-1" library="supply1" deviceset="V-" device=""/>
 <part name="P-3" library="supply1" deviceset="V-" device=""/>
-<part name="C1" library="rcl" deviceset="C-EU" device="C0603"/>
-<part name="R1" library="rcl" deviceset="R-EU_" device="R0603"/>
-<part name="R2" library="rcl" deviceset="R-EU_" device="R0603"/>
-<part name="C2" library="rcl" deviceset="C-EU" device="C0603"/>
-<part name="R3" library="rcl" deviceset="R-EU_" device="R0603"/>
-<part name="R4" library="rcl" deviceset="R-EU_" device="R0603"/>
-<part name="C3" library="rcl" deviceset="C-EU" device="C0603"/>
-<part name="C4" library="rcl" deviceset="C-EU" device="C0603"/>
-<part name="R5" library="rcl" deviceset="R-EU_" device="R0603"/>
-<part name="R6" library="rcl" deviceset="R-EU_" device="R0603"/>
+<part name="C1" library="rcl" deviceset="C-EU" device="C0603" value="100n"/>
+<part name="R1" library="rcl" deviceset="R-EU_" device="R0603" value="49R9"/>
+<part name="R2" library="rcl" deviceset="R-EU_" device="R0603" value="49R9"/>
+<part name="C2" library="rcl" deviceset="C-EU" device="C0603" value="100p"/>
+<part name="R3" library="rcl" deviceset="R-EU_" device="R0603" value="470"/>
+<part name="R4" library="rcl" deviceset="R-EU_" device="R0603" value="470"/>
+<part name="C3" library="rcl" deviceset="C-EU" device="C0603" value="DNP"/>
+<part name="C4" library="rcl" deviceset="C-EU" device="C0603" value="DNP"/>
+<part name="R5" library="rcl" deviceset="R-EU_" device="R0603" value="470"/>
+<part name="R6" library="rcl" deviceset="R-EU_" device="R0603" value="470"/>
 <part name="GND1" library="supply1" deviceset="GND" device=""/>
 <part name="K1" library="relay" deviceset="FTR-B4" device="G"/>
@@
 <part name="P+3" library="supply1" deviceset="V+" device=""/>
 <part name="P-2" library="supply1" deviceset="V-" device=""/>
-<part name="C7" library="rcl" deviceset="C-EU" device="C0603"/>
-<part name="R15" library="rcl" deviceset="R-EU_" device="R0603"/>
-<part name="R16" library="rcl" deviceset="R-EU_" device="R0603"/>
-<part name="C8" library="rcl" deviceset="C-EU" device="C0603"/>
-<part name="R17" library="rcl" deviceset="R-EU_" device="R0603"/>
-<part name="R18" library="rcl" deviceset="R-EU_" device="R0603"/>
-<part name="C9" library="rcl" deviceset="C-EU" device="C0603"/>
-<part name="C10" library="rcl" deviceset="C-EU" device="C0603"/>
-<part name="R19" library="rcl" deviceset="R-EU_" device="R0603"/>
-<part name="R20" library="rcl" deviceset="R-EU_" device="R0603"/>
+<part name="C7" library="rcl" deviceset="C-EU" device="C0603" value="100n"/>
+<part name="R15" library="rcl" deviceset="R-EU_" device="R0603" value="49R9"/>
+<part name="R16" library="rcl" deviceset="R-EU_" device="R0603" value="49R9"/>
+<part name="C8" library="rcl" deviceset="C-EU" device="C0603" value="100p"/>
+<part name="R17" library="rcl" deviceset="R-EU_" device="R0603" value="470"/>
+<part name="R18" library="rcl" deviceset="R-EU_" device="R0603" value="470"/>
+<part name="C9" library="rcl" deviceset="C-EU" device="C0603" value="DNP"/>
+<part name="C10" library="rcl" deviceset="C-EU" device="C0603" value="DNP"/>
+<part name="R19" library="rcl" deviceset="R-EU_" device="R0603" value="470"/>
+<part name="R20" library="rcl" deviceset="R-EU_" device="R0603" value="470"/>
 <part name="GND8" library="supply1" deviceset="GND" device=""/>
 <part name="X3" library="con-coax" deviceset="?227161*" device="1-" technology="-7" value="1-1337543-0"/>
@@
 <part name="C19" library="rcl" deviceset="C-EU" device="C0603" value="1u"/>
 <part name="GND21" library="supply1" deviceset="GND" device=""/>
-<part name="L1" library="rcl" deviceset="L-EU" device="L2012C"/>
+<part name="L1" library="rcl" deviceset="L-EU" device="L2012C" value="Ferrite"/>
 <part name="C20" library="rcl" deviceset="C-EU" device="C1206" value="10u"/>
 <part name="C21" library="rcl" deviceset="C-EU" device="C1206" value="10u"/>
-<part name="L2" library="rcl" deviceset="L-EU" device="L2012C"/>
+<part name="L2" library="rcl" deviceset="L-EU" device="L2012C" value="Ferrite"/>
 <part name="C22" library="rcl" deviceset="C-EU" device="C1206" value="10u"/>
 <part name="C23" library="rcl" deviceset="C-EU" device="C1206" value="10u"/>
@@
 <instance part="C4" gate="G$1" x="180.34" y="121.92" smashed="yes" rot="R90">
 <attribute name="NAME" x="184.404" y="119.761" size="1.778" layer="95"/>
-<attribute name="VALUE" x="185.039" y="123.444" size="1.778" layer="96" rot="R90"/>
+<attribute name="VALUE" x="188.976" y="124.079" size="1.778" layer="96" rot="R180"/>
 </instance>
 <instance part="R5" gate="G$1" x="160.02" y="144.78" smashed="yes">
 <attribute name="NAME" x="156.21" y="146.2786" size="1.778" layer="95"/>
-<attribute name="VALUE" x="156.21" y="141.478" size="1.778" layer="96"/>
+<attribute name="VALUE" x="161.29" y="146.558" size="1.778" layer="96"/>
 </instance>
 <instance part="R6" gate="G$1" x="160.02" y="139.7" smashed="yes">
 <attribute name="NAME" x="156.21" y="141.1986" size="1.778" layer="95"/>
-<attribute name="VALUE" x="156.21" y="136.398" size="1.778" layer="96"/>
+<attribute name="VALUE" x="161.29" y="141.478" size="1.778" layer="96"/>
 </instance>
 <instance part="GND1" gate="1" x="200.66" y="127" smashed="yes">
@@
 <instance part="C9" gate="G$1" x="180.34" y="114.3" smashed="yes" rot="R90">
 <attribute name="NAME" x="179.959" y="115.824" size="1.778" layer="95" rot="R90"/>
-<attribute name="VALUE" x="185.039" y="115.824" size="1.778" layer="96" rot="R90"/>
+<attribute name="VALUE" x="184.404" y="114.681" size="1.778" layer="96"/>
 </instance>
 <instance part="C10" gate="G$1" x="180.34" y="73.66" smashed="yes" rot="R90">
 <attribute name="NAME" x="184.404" y="71.501" size="1.778" layer="95"/>
-<attribute name="VALUE" x="185.039" y="75.184" size="1.778" layer="96" rot="R90"/>
+<attribute name="VALUE" x="184.404" y="74.041" size="1.778" layer="96"/>
 </instance>
 <instance part="R19" gate="G$1" x="160.02" y="96.52" smashed="yes">
 <attribute name="NAME" x="156.21" y="98.0186" size="1.778" layer="95"/>
-<attribute name="VALUE" x="156.21" y="93.218" size="1.778" layer="96"/>
+<attribute name="VALUE" x="161.29" y="98.298" size="1.778" layer="96"/>
 </instance>
 <instance part="R20" gate="G$1" x="160.02" y="91.44" smashed="yes">
 <attribute name="NAME" x="156.21" y="92.9386" size="1.778" layer="95"/>
-<attribute name="VALUE" x="156.21" y="88.138" size="1.778" layer="96"/>
+<attribute name="VALUE" x="161.29" y="93.218" size="1.778" layer="96"/>
 </instance>
 <instance part="GND8" gate="1" x="200.66" y="78.74" smashed="yes">
@@
 </sheet>
 </sheets>
+<errors>
+</errors>
 </schematic>
 </drawing>

Commit message: Added testpoints, changes to silkscreen, created Gerber
Parts:
- added TP1, TP2, TP3: TPTP15R, testpad:TPTP15R
Connections:
- net GND: now also IC5.SDIN/FORMAT, TP2.TP
- net V+: now also TP1.TP; no longer IC5.SDIN/FORMAT
- net V-: now also TP3.TP
Other:
- note added: "Jumper cable: Molex 15166-0214"

Commit message: Part values corrected
Parts:
- C10, C3, C4, C9: value DNP -> 33p
- R11, R25: value 750k -> 750k||18p
- R12, R26: value 190k -> 190k||68p
- R13, R27: value 60k -> 60k||220p
- R14, R28: value 10k -> 1k
